File: incubator_buttom.kicad_pcb (KiCad board)
At the start: 2 copper layers, 22 parts, among them J1 CONTORL, SW1 STOP_PHOTO, SW2 HUMIDITY, SW3 STOP_INCUBATOR, SW4 START_PHOTO, SW5 START_INCUBATOR

Commit message: complete
Parts:
- added C10: 0.1MIF, Capacitor_THT:C_Disc_D3.0mm_W1.6mm_P2.50mm, F.Cu at (124.0, 73.2)
- added C7: 0.1MIF, Capacitor_THT:C_Disc_D3.0mm_W1.6mm_P2.50mm, F.Cu at (88.9, 49.8)
- added C8: 0.1MIF, Capacitor_THT:C_Disc_D3.0mm_W1.6mm_P2.50mm, F.Cu at (121.9, 53.1)
- added C9: 0.1MIF, Capacitor_THT:C_Disc_D3.0mm_W1.6mm_P2.50mm, F.Cu at (107.4, 36.3)
- R1, R10, R2, R3, R4, R5, R6, R7, R8, R9: footprint Resistor_THT:R_Axial_DIN0204_L3.6mm_D1.6mm_P5.08mm_Horizontal -> Resistor_THT:R_Axial_DIN0207_L6.3mm_D2.5mm_P10.16mm_Horizontal
- moved SW5 73.4 mm to (112.2, 36.7)
- moved R10 63.5 mm to (119.4, 47.2), turned to 180 degrees
- moved C5 63.2 mm to (122.2, 47.2), turned to 0 degrees
- moved SW3 59.8 mm to (89.7, 36.7)
- moved R6 50.7 mm to (101.9, 47.8), turned to 180 degrees
- moved C3 47.9 mm to (101.9, 50.8), turned to 0 degrees
- moved R9 47.5 mm to (109.2, 50.5), turned to 0 degrees
- moved SW4 43.3 mm to (112.2, 59.7)
- moved C4 41.6 mm to (126.5, 70.1), turned to 180 degrees
- moved R5 40.9 mm to (99.1, 52.8), turned to 180 degrees
- moved SW2 31.8 mm to (101.2, 81.7)
- moved R8 29.5 mm to (111.3, 70.4), turned to 0 degrees
- moved R7 27.0 mm to (111.3, 73.7), turned to 0 degrees
- moved C2 25.1 mm to (125.2, 83.1), turned to 180 degrees
- moved R4 24.3 mm to (127.3, 80.0), turned to 180 degrees
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Connections:
- C1 pad 1: /GND -> Net-(C1-Pad1)
- C1 pad 2: /MC2 -> /GND
- C2 pad 1: /GND -> Net-(C2-Pad1)
- C2 pad 2: /MC3 -> /GND
- C3 pad 1: /GND -> Net-(C3-Pad1)
- C3 pad 2: /MC4 -> /GND
- C4 pad 2: /MC1 -> Net-(C4-Pad2)
- C5 pad 1: /GND -> Net-(C5-Pad1)
- C5 pad 2: /MC5 -> /GND
- R10 pad 1: /MC5 -> Net-(C5-Pad1)
- R10 pad 2: Net-(R10-Pad2) -> /MC5
- R2 pad 2: Net-(R2-Pad2) -> Net-(C1-Pad1)
- R4 pad 1: /MC3 -> Net-(C2-Pad1)
- R4 pad 2: Net-(R4-Pad2) -> /MC3
- R6 pad 1: /MC4 -> Net-(C3-Pad1)
- R6 pad 2: Net-(R6-Pad2) -> /MC4
- R8 pad 2: Net-(R8-Pad2) -> Net-(C4-Pad2)
- SW1 pad 2: Net-(R2-Pad2) -> /MC2
- SW2 pad 2: Net-(R4-Pad2) -> /MC3
- SW3 pad 2: Net-(R6-Pad2) -> /MC4
- SW4 pad 2: Net-(R8-Pad2) -> /MC1
- SW5 pad 2: Net-(R10-Pad2) -> /MC5
Routing:
- net /MC2: track 18.5 -> 48.4 mm
- net /VCC: track 230.7 -> 255.5 mm
- net /MC3: track 12.2 -> 35.6 mm
- net /MC1: track 23.4 -> 46.4 mm
- net /MC4: track 58.1 -> 79.5 mm
- net Net-(R4-Pad2): track 19.6 -> 0.00 mm
- net Net-(R10-Pad2): track 18.8 -> 0.00 mm
- net Net-(R8-Pad2): track 18.6 -> 0.00 mm
- net Net-(R6-Pad2): track 16.5 -> 0.00 mm
- net Net-(R2-Pad2): track 16.0 -> 0.00 mm
- net /MC5: track 49.2 -> 63.1 mm
- net /GND: track 62.5 -> 50.1 mm
- net Net-(C2-Pad1): track 0.00 -> 3.89 mm
- net Net-(C3-Pad1): track 0.00 -> 3.05 mm
- net Net-(C5-Pad1): track 0.00 -> 2.79 mm
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