File: incubator_buttom.sch (KiCad schematic (older format))
At the start: 22 parts, among them J1 CONTORL, SW1 STOP_PHOTO, SW2 HUMIDITY, SW3 STOP_INCUBATOR, SW4 START_PHOTO, SW5 START_INCUBATOR

Commit message: complete
Parts:
- added C10, C7, C8, C9: 0.1MIF, Capacitor_THT:C_Disc_D3.0mm_W1.6mm_P2.50mm, symbol Device:C
- R1, R10, R2, R3, R4, R5, R6, R7, R8, R9: footprint Resistor_THT:R_Axial_DIN0204_L3.6mm_D1.6mm_P5.08mm_Horizontal -> Resistor_THT:R_Axial_DIN0207_L6.3mm_D2.5mm_P10.16mm_Horizontal
Connections:
- net GND: now also C1.2, C2.2, C3.2, C5.2, C10.2, C7.2, C8.2, C9.2; no longer C1.1, C2.1, C3.1, C5.1
- net MC2: now also SW1.2; no longer C1.2
- net MC3: now also R4.2, SW2.2; no longer C2.2, R4.1
- net MC4: now also R6.2, SW3.2; no longer C3.2, R6.1
- net MC5: now also R10.2, SW5.2; no longer C5.2, R10.1
- net VCC: now also C10.1, C7.1, C8.1, C9.1
- net at R2.2: now also C1.1; no longer SW1.2
- new net: C2.1, R4.1
- new net: C3.1, R6.1
- new net: C5.1, R10.1
Other:
- moved on the sheet: C1, C2, C3, C4, C5, C6, J1, R1, R10, R2, R3, R4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
